File: hw/_autosave-baseline_project.kicad_sch (KiCad schematic)
At the start: 20 parts, among them J101 EXT_3V3, Q101 IRLD024PBF, SW101 UP, SW102 DOWN, SW103 LEFT, SW104 RIGHT, SW105 MODE, U101 EK-TM4C123GXL, U102 ESP8266-1, U103 Adafruit ST7735R

Commit message: Speaker
Parts:
- added R1: 10k, ECE445L:R_Axial_DIN0204_L3.6mm_D1.6mm_P7.62mm_Horizontal, symbol ECE445L:R_0.125W
- added SW1: Select, Button_Switch_THT:SW_PUSH_6mm, symbol Switch:SW_Push
Connections:
- net +3V3: now also SW1.2
- net GND: now also R1.2
- net PF0: now also R1.1, SW1.1

Commit message: Speaker + Thermistor
Parts:
- added R2: 10k, ECE445L:R_Axial_DIN0204_L3.6mm_D1.6mm_P7.62mm_Horizontal, symbol ECE445L:R_0.125W
- added TH1: Thermistor_US, symbol Device:Thermistor_US
Connections:
- net +3V3: now also R2.1
- net GND: now also TH1.2
- net PE4: now also R2.2, TH1.1

Commit message: Alarm Functioning
Parts:
- added RV1: R_Potentiometer, symbol Device:R_Potentiometer
Connections:
- net +3V3: now also RV1.1
- net GND: now also RV1.3
- net PE3: now also RV1.2
